Commit message: Fix mass spring dynamics
Fixed incorrect calculation of mass spring forces and incorrect geometry, refactored simulation module code

File: elevator.urdf (robot description, URDF)
Before this commit: robot elevator, 6 links, 5 joints
Links:
- link elevator: mass 0.1 -> .1
- link frame_end: mass None -> 0.0001
- link frame_hor: mass 0.1 -> .1
- link frame_ver: mass 0.1 -> .1
- link prism_rod: geometry collision cylinder length=0.09 radius=0.01; visual cylinder length=0.09 radius=0.01
Joints:
- joint elevatortorod: limit lower=0.0 upper=.01 -> lower=0.0 upper=.1

File: lever.urdf (robot description, URDF)
Before this commit: robot lever, 3 links, 2 joints
Links:
- link lever: mass 1.0 -> .1
- link lever_end: mass None -> 0.0001
Joints:
- joint basetolever: limit lower=-0.3 upper=0.3 effort=10.0 velocity=10.0 -> lower=-1.0472 upper=1.0472
- joint possensor: origin xyz=-0.001 0.0 -0.3 -> xyz=-0.01 0.0 -0.2
